Commit message: working for pips controler and collision checking with realsense.

File: robots/pioneer3at_realsense.xacro (robot description, xacro)
@@ -4,5 +4,5 @@
        xmlns:interface="http://playerstage.sourceforge.net/gazebo/xmlschema/#interface"
        xmlns:xacro="http://ros.org/wiki/xacro"
-name="pioneer3at"
+name="pioneer"
 >
 <!-- Chassis -->
@@ -78,5 +78,5 @@
     </gazebo>
     <joint name="base_top_joint" type="fixed">
-        <origin xyz="0.003 0 0.274" rpy="0 0 0"/>
+        <origin xyz="0.035 0 0.274" rpy="0 0 0"/>
         <parent link="base_link"/>
         <child link="top_plate"/>
@@ -431,70 +431,9 @@
     <odometryTopic>odom</odometryTopic>
     <odometryFrame>odom</odometryFrame>
-    <covarianc_x> 0.001</covariance_x>
+    <covariance_x> 0.001</covariance_x>
     <covariance_y>0.001</covariance_y>
     <covariance_yaw>0.01</covariance_yaw>
     <broadcastTF>1</broadcastTF>
   </plugin>
-</gazebo>
-<joint name="hokuyo_joint" type="fixed">
-    <axis xyz="0 1 0" />
-    <origin xyz="0.150 0 0.037" rpy="0 0 0"/>
-    <parent link="top_plate"/>
-    <child link="hokuyo_link"/>
-</joint>
-  <!-- Hokuyo Laser -->
-  <link name="hokuyo_link">
-    <collision>
-      <origin xyz="0 0 0" rpy="0 0 0"/>
-      <geometry>
-    <box size="0.01 0.01 0.01"/>
-      </geometry>
-    </collision>
-    <visual>
-      <origin xyz="0 0 0" rpy="0 0 0"/>
-      <geometry>
-        <mesh filename="package://p3at_tutorial/meshes/hokuyo1.dae"/>
-      </geometry>
-    </visual>
-    <inertial>
-      <mass value="1e-5" />
-      <origin xyz="0 0 0" rpy="0 0 0"/>
-      <inertia ixx="1e-6" ixy="0" ixz="0" iyy="1e-6" iyz="0" izz="1e-6" />
-    </inertial>
-  </link>
-<gazebo reference="hokuyo_link">
-    <sensor type="ray" name="head_hokuyo_sensor">
-      <pose>0 0 0 0 0 0</pose>
-      <visualize>true</visualize>
-      <update_rate>40</update_rate>
-      <ray>
-        <scan>
-          <horizontal>
-            <samples>1080</samples>
-            <resolution>1</resolution>
-            <min_angle>-2.3559777</min_angle>
-            <max_angle>2.3559777</max_angle>
-          </horizontal>
-        </scan>
-        <range>
-          <min>0.10</min>
-          <max>30.0</max>
-          <resolution>0.01</resolution>
-        </range>
-        <noise>
-          <type>gaussian</type>
-          <!-- Noise parameters based on published spec for Hokuyo laser
-               achieving "+-30mm" accuracy at range < 10m.  A mean of 0.0m and
-               stddev of 0.01m will put 99.7% of samples within 0.03m of the true
-               reading. -->
-          <mean>0.0</mean>
-          <stddev>0.01</stddev>
-        </noise>
-      </ray>
-      <plugin name="gazebo_ros_head_hokuyo_controller" filename="libgazebo_ros_laser.so">
-        <topicName>/hokuyo_scan</topicName>
-        <frameName>hokuyo_link</frameName>
-      </plugin>
-    </sensor>
 </gazebo>
 <gazebo reference="front_sonar">
@@ -595,4 +534,176 @@
 <!-- <xacro:p3at_back suffix="left" reflect="1"/> -->
 <!-- <xacro:p3at_back suffix="right" reflect="-1"/> -->
-<xacro:p3at_gazebo_ext/>
+ <!-- Camera link -->
+    <link name="rs200_camera">
+        <visual>
+            <origin rpy="0 0 0" xyz="0 0 0"/>
+            <geometry>
+                <mesh filename="package://realsense_gazebo_plugin/models/realsense_camera/meshes/realsense.dae"/>
+            </geometry>
+        </visual>
+        <collision>
+            <geometry>
+                <box size="0.0078 0.130 0.0192"/>
+            </geometry>
+        </collision>
+        <inertial>
+            <mass value="0.0615752"/>
+            <origin rpy="0 0 0" xyz="0 0 0"/>
+            <inertia ixx="9.108e-05"
+                     ixy="0"
+                     ixz="0"
+                     iyy="2.51e-06"
+                     iyz="0"
+                     izz="8.931e-05"
+            />
+        </inertial>
+    </link>
+    <!-- Virtual links representing the cameras positons and orientations-->
+    <link name="color" />
+    <link name="depth" />
+    <link name="ired1" />
+    <link name="ired2" />
+    <!-- Joints positioning the virtual links with respect to the camera main link-->
+    <joint name="color_joint" type="fixed">
+        <parent link="rs200_camera" />
+        <child link="color" />
+        <!-- <origin xyz="0 -0.046 0.004" rpy="0 0 0"/> -->
+        <!-- The default position is change since in Rviz the cloud depth axis is Z not X-->
+        <origin xyz="0 -0.046 0.004" rpy="${pi/2} ${pi} ${pi/2}"/>
+    </joint>
+    <joint name="depth_joint" type="fixed">
+        <parent link="rs200_camera" />
+        <child link="depth" />
+        <origin xyz="0 -0.03 0.004" rpy="0 0 0"/>
+    </joint>
+    <joint name="ired1_joint" type="fixed">
+        <parent link="rs200_camera" />
+        <child link="ired1" />
+        <origin xyz="0 -0.06 0.004" rpy="0 0 0"/>
+    </joint>
+    <joint name="ired2_joint" type="fixed">
+        <parent link="rs200_camera" />
+        <child link="ired2" />
+        <origin xyz="0 0.01 0.004" rpy="0 0 0"/>
+    </joint>
+  <joint name="base_real" type="fixed">
+	<origin xyz="0.25 0 0.24" rpy="0 0 0"/>
+	<parent link="base_link"/>
+	<child link="rs200_camera"/>
+  </joint>
+<!-- **********************************************************-->
+<!-- GAZEBO DEFINITIONS ***************************************-->
+    <!-- Load plugin to the model ("robot" in urdf format)-->
+    <gazebo>
+        <plugin name="realsense_plugin" filename="librealsense_gazebo_plugin.so"/>
+        <!--<pose frame="">0 0 0.015 0 0 0</pose>-->
+    </gazebo>
+    <!-- Load parameters to model's main link-->
+    <gazebo reference="rs200_camera">
+        <self_collide>0</self_collide>
+        <enable_wind>0</enable_wind>
+        <kinematic>0</kinematic>
+        <gravity>1</gravity>
+        <!--<mu>1</mu>-->
+        <mu2>1</mu2>
+        <fdir1>0 0 0</fdir1>
+        <!--<slip1>0</slip1>
+        <slip2>0</slip2>-->
+        <kp>1e+13</kp>
+        <kd>1</kd>
+        <!--<max_vel>0.01</max_vel>
+        <min_depth>0</min_depth>-->
+        <sensor name="color" type="camera">
+            <pose frame="">0 -0.046 0.004 0 0 0</pose>
+            <camera name="__default__">
+            <horizontal_fov>1.047</horizontal_fov>
+            <image>
+                <width>640</width>
+                <height>480</height>
+                <format>RGB_INT8</format>
+            </image>
+            <clip>
+                <near>0.1</near>
+                <far>100</far>
+            </clip>
+            <noise>
+                <type>gaussian</type>
+                <mean>0.0</mean>
+                <stddev>0.007</stddev>
+            </noise>
+            </camera>
+            <always_on>1</always_on>
+            <update_rate>60</update_rate>
+            <visualize>1</visualize>
+        </sensor>
+        <sensor name="ired1" type="camera">
+            <pose frame="">0 -0.06 0.004 0 0 0</pose>
+            <camera name="__default__">
+            <horizontal_fov>1.047</horizontal_fov>
+            <image>
+                <width>640</width>
+                <height>480</height>
+                <format>L_INT8</format>
+            </image>
+            <clip>
+                <near>0.1</near>
+                <far>100</far>
+            </clip>
+            <noise>
+                <type>gaussian</type>
+                <mean>0.0</mean>
+                <stddev>0.05</stddev>
+            </noise>
+            </camera>
+            <always_on>1</always_on>
+            <update_rate>60</update_rate>
+            <visualize>0</visualize>
+        </sensor>
+        <sensor name="ired2" type="camera">
+            <pose frame="">0 0.01 0.004 0 0 0</pose>
+            <camera name="__default__">
+            <horizontal_fov>1.047</horizontal_fov>
+            <image>
+                <width>640</width>
+                <height>480</height>
+                <format>L_INT8</format>
+            </image>
+            <clip>
+                <near>0.1</near>
+                <far>100</far>
+            </clip>
+            <noise>
+                <type>gaussian</type>
+                <mean>0.0</mean>
+                <stddev>0.05</stddev>
+            </noise>
+            </camera>
+            <always_on>1</always_on>
+            <update_rate>60</update_rate>
+            <visualize>0</visualize>
+        </sensor>
+        <sensor name="depth" type="depth">
+            <pose frame="">0 -0.03 0.004 0 0 0</pose>
+            <camera name="__default__">
+            <horizontal_fov>1.047</horizontal_fov>
+            <image>
+                    <width>640</width>
+                    <height>480</height>
+            </image>
+            <clip>
+                    <near>0.1</near>
+                    <far>100</far>
+            </clip>
+            <noise>
+                    <type>gaussian</type>
+                    <mean>0.0</mean>
+                    <stddev>0.100</stddev>
+            </noise>
+            </camera>
+            <always_on>1</always_on>
+            <update_rate>60</update_rate>
+            <visualize>0</visualize>
+        </sensor>
+    </gazebo>
+    <xacro:p3at_gazebo_ext/>
 </robot>
