Commit message: Clean the robots files, add stereo. The robot can be rendered in the gazebo.

File: robots/pioneer3at.xacro (robot description, xacro)
@@ -6,4 +6,5 @@
 name="pioneer3at"
 >
+<xacro:property name="M_PI" value="3.1415926535897931" />
 <!-- Chassis -->
     <link name="base_link">
@@ -431,70 +432,9 @@
     <odometryTopic>odom</odometryTopic>
     <odometryFrame>odom</odometryFrame>
-    <covarianc_x> 0.001</covariance_x>
+    <covariance_x> 0.001</covariance_x>
     <covariance_y>0.001</covariance_y>
     <covariance_yaw>0.01</covariance_yaw>
     <broadcastTF>1</broadcastTF>
   </plugin>
-</gazebo>
-<joint name="hokuyo_joint" type="fixed">
-    <axis xyz="0 1 0" />
-    <origin xyz="0.150 0 0.037" rpy="0 0 0"/>
-    <parent link="top_plate"/>
-    <child link="hokuyo_link"/>
-</joint>
-  <!-- Hokuyo Laser -->
-  <link name="hokuyo_link">
-    <collision>
-      <origin xyz="0 0 0" rpy="0 0 0"/>
-      <geometry>
-    <box size="0.01 0.01 0.01"/>
-      </geometry>
-    </collision>
-    <visual>
-      <origin xyz="0 0 0" rpy="0 0 0"/>
-      <geometry>
-        <mesh filename="package://p3at_tutorial/meshes/hokuyo1.dae"/>
-      </geometry>
-    </visual>
-    <inertial>
-      <mass value="1e-5" />
-      <origin xyz="0 0 0" rpy="0 0 0"/>
-      <inertia ixx="1e-6" ixy="0" ixz="0" iyy="1e-6" iyz="0" izz="1e-6" />
-    </inertial>
-  </link>
-<gazebo reference="hokuyo_link">
-    <sensor type="ray" name="head_hokuyo_sensor">
-      <pose>0 0 0 0 0 0</pose>
-      <visualize>true</visualize>
-      <update_rate>40</update_rate>
-      <ray>
-        <scan>
-          <horizontal>
-            <samples>1080</samples>
-            <resolution>1</resolution>
-            <min_angle>-2.3559777</min_angle>
-            <max_angle>2.3559777</max_angle>
-          </horizontal>
-        </scan>
-        <range>
-          <min>0.10</min>
-          <max>30.0</max>
-          <resolution>0.01</resolution>
-        </range>
-        <noise>
-          <type>gaussian</type>
-          <!-- Noise parameters based on published spec for Hokuyo laser
-               achieving "+-30mm" accuracy at range < 10m.  A mean of 0.0m and
-               stddev of 0.01m will put 99.7% of samples within 0.03m of the true
-               reading. -->
-          <mean>0.0</mean>
-          <stddev>0.01</stddev>
-        </noise>
-      </ray>
-      <plugin name="gazebo_ros_head_hokuyo_controller" filename="libgazebo_ros_laser.so">
-        <topicName>/hokuyo_scan</topicName>
-        <frameName>hokuyo_link</frameName>
-      </plugin>
-    </sensor>
 </gazebo>
 <gazebo reference="front_sonar">

File: robots/pioneer3at_realsense.xacro (robot description, xacro)
@@ -4,534 +4,7 @@
        xmlns:interface="http://playerstage.sourceforge.net/gazebo/xmlschema/#interface"
        xmlns:xacro="http://ros.org/wiki/xacro"
-name="pioneer"
+name="pioneer3at"
 >
-<!-- Chassis -->
-    <link name="base_link">
-        <inertial>
-            <mass value="10.0"/>
-            <origin xyz="0 0 0.177"/>
-            <inertia ixx="0.3338" ixy="0.0" ixz="0.0"
-                 iyy="0.4783" iyz="0.0"
-                 izz="0.3338"/>
-        </inertial>
-        <visual name="base_visual">
-            <origin xyz="0 0 0.177" rpy="0 0 0"/>
-            <geometry name="pioneer_geom">
-                <mesh filename="package://p3at_tutorial/meshes/p3at_meshes/chassis.dae"/>
-            </geometry>
-            <material name="ChassisRed">
-                <color rgba="0.851 0.0 0.0 1.0"/>
-            </material>
-        </visual>
-        <collision>
-            <origin xyz="0 0 0.177" rpy="0 0 0"/>
-                <geometry>
-                    <mesh filename="package://p3at_tutorial/meshes/p3at_meshes/chassis.dae"/>
-                </geometry>
-        </collision>
-    </link>
-    <gazebo reference="base_link">
-        <material value="Gazebo/Red"/>
-    </gazebo>
-<!--link name="odom">
-</link>
-<joint name="odom_base" type="floating">
-        <origin xyz="0 0 0" rpy="0 0 0"/>
-        <parent link="odom"/>
-        <child link="base_link"/>
-    </joint-->
-<!--<link name="map">
-</link-->
-<!--<joint name="map_odom" type="fixed">
-        <origin xyz="0 0 0" rpy="0 0 0"/>
-        <parent link="map"/>
-        <child link="odom"/>
-    </joint>
-    -->
-<!-- Top -->
-    <link name="top_plate">
-        <inertial>
-            <mass value="0.1"/>
-            <origin xyz="-0.025 0 -0.223"/>
-            <inertia ixx="1.0" ixy="0.0" ixz="0.0"
-                 iyy="1.0" iyz="0.0"
-                izz="1.0"/>
-        </inertial>
-        <visual name="base_visual">
-            <origin xyz="0 0 0" rpy="0 0 0"/>
-            <geometry name="pioneer_geom">
-                <mesh filename="package://p3at_tutorial/meshes/p3at_meshes/top.dae"/>
-            </geometry>
-            <material name="TopBlack">
-                    <color rgba="0.038 0.038 0.038 1.0"/>
-            </material>
-        </visual>
-        <collision>
-            <origin xyz="0 0 0" rpy="0 0 0"/>
-            <geometry>
-                <box size="0.01 0.01 0.01"/>
-            </geometry>
-        </collision>
-    </link>
-    <gazebo reference="top_plate">
-        <material value="Gazebo/Black"/>
-    </gazebo>
-    <joint name="base_top_joint" type="fixed">
-        <origin xyz="0.035 0 0.274" rpy="0 0 0"/>
-        <parent link="base_link"/>
-        <child link="top_plate"/>
-    </joint>
-<!-- Front + Back Sonar -->
-    <link name="front_sonar">
-        <inertial>
-            <mass value="0.1"/>
-            <origin xyz="0 0 0"/>
-            <inertia ixx="1.0" ixy="0.0" ixz="0.0"
-                 iyy="1.0" iyz="0.0" izz="1.0"/>
-        </inertial>
-        <visual name="base_visual">
-            <origin xyz="0 0 0" rpy="0 0 0"/>
-            <geometry name="pioneer_geom">
-                <mesh filename="package://p3at_tutorial/meshes/p3at_meshes/front_sonar.dae"/>
-            </geometry>
-            <material name="SonarYellow">
-                <color rgba="0.715 0.583 0.210 1.0"/>
-            </material>
-        </visual>
-        <collision>
-            <origin xyz="0 0 0" rpy="0 0 0"/>
-            <geometry>
-                <box size="0.01 0.01 0.01"/>
-            </geometry>
-        </collision>
-    </link>
-    <gazebo reference="front_sonar">
-        <material value="Gazebo/Yellow"/>
-    </gazebo>
-    <joint name="base_front_joint" type="fixed">
-        <origin xyz="0.193 0 0.25" rpy="0 0 0"/>
-        <parent link="base_link"/>
-        <child link="front_sonar"/>
-    </joint>
-    <link name="back_sonar">
-        <inertial>
-            <mass value="0.1"/>
-            <origin xyz="0 0 0"/>
-            <inertia ixx="1.0" ixy="0.0" ixz="0.0"
-                 iyy="1.0" iyz="0.0" izz="1.0"/>
-        </inertial>
-        <visual name="base_visual">
-            <origin xyz="0 0 0" rpy="0 0 0"/>
-            <geometry name="pioneer_geom">
-                <mesh filename="package://p3at_tutorial/meshes/p3at_meshes/back_sonar.dae"/>
-            </geometry>
-            <material name="SonarYellow">
-                <color rgba="0.715 0.583 0.210 1.0"/>
-            </material>
-        </visual>
-        <collision>
-            <origin xyz="0 0 0" rpy="0 0 0"/>
-            <geometry>
-                <box size="0.01 0.01 0.01"/>
-            </geometry>
-        </collision>
-    </link>
-    <gazebo reference="back_sonar">
-        <material value="Gazebo/Yellow"/>
-    </gazebo>
-    <joint name="base_back_joint" type="fixed">
-        <origin xyz="-0.187 0 0.247" rpy="0 0 0"/>
-        <parent link="base_link"/>
-        <child link="back_sonar"/>
-    </joint>
-<link name="back_sonar_fake">
-    <inertial>
-            <mass value="0.1"/>
-            <origin xyz="0 0 0"/>
-            <inertia ixx="1.0" ixy="0.0" ixz="0.0"
-                 iyy="1.0" iyz="0.0" izz="1.0"/>
-    </inertial>
-<!--     <visual name="base_visual">
-            <origin xyz="0 0 0" rpy="0 0 0"/>
-            <geometry name="pioneer_geom">
-                <mesh filename="package://p3at_tutorial/meshes/p3at_meshes/back_sonar.dae"/>
-            </geometry>
-            <material name="SonarYellow">
-                <color rgba="0.715 0.583 0.210 1.0"/>
-            </material>
-        </visual>
-        <collision>
-            <origin xyz="0 0 0" rpy="0 0 0"/>
-            <geometry>
-                <box size="0.01 0.01 0.01"/>
-            </geometry>
-        </collision> -->
-</link>
-<joint name="base_back_sonar_joint" type="fixed">
-    <origin xyz="0 0 0" rpy="0 0 3.1415"/>
-    <parent link="back_sonar"/>
-    <child link="back_sonar_fake"/>
-</joint>
-<link name="imu">
-    <inertial>
-            <mass value="0.1"/>
-            <origin xyz="0 0 0"/>
-            <inertia ixx="1.0" ixy="0.0" ixz="0.0"
-                 iyy="1.0" iyz="0.0" izz="1.0"/>
-    </inertial>
-<!--     <visual name="base_visual">
-            <origin xyz="0 0 0" rpy="0 0 0"/>
-            <geometry name="pioneer_geom">
-                <mesh filename="package://p3at_tutorial/meshes/p3at_meshes/back_sonar.dae"/>
-            </geometry>
-            <material name="SonarYellow">
-                <color rgba="0.715 0.583 0.210 1.0"/>
-            </material>
-        </visual>
-        <collision>
-            <origin xyz="0 0 0" rpy="0 0 0"/>
-            <geometry>
-                <box size="0.01 0.01 0.01"/>
-            </geometry>
-        </collision> -->
-</link>
-<joint name="imu_joint" type="fixed">
-    <origin xyz="0 0 0" rpy="3.1415 0 0"/>
-    <parent link="base_link"/>
-    <child link="imu"/>
-</joint>
-<!-- Front Axles + Wheels + Hubcaps -->
-<xacro:macro name="p3at_front" params="suffix reflect">
-    <link name="p3at_front_${suffix}_axle">
-        <inertial>
-            <mass value="0.1"/>
-            <origin xyz="0 0 0"/>
-            <inertia ixx="1.0" ixy="0.0" ixz="0.0"
-                 iyy="1.0" iyz="0.0" izz="1.0"/>
-        </inertial>
-    <visual name="base_visual">
-        <origin xyz="0 0 0" rpy="0 0 0"/>
-        <geometry name="pioneer_geom">
-            <mesh filename="package://p3at_tutorial/meshes/p3at_meshes/axle.dae"/>
-        </geometry>
-        <material name="AxleGrey">
-            <color rgba="0.5 0.5 0.5 1"/>
-        </material>
-    </visual>
-    <collision>
-        <origin xyz="0 0 0" rpy="0 0 0"/>
-        <geometry>
-            <box size="0.01 0.01 0.01"/>
-        </geometry>
-    </collision>
-    </link>
-    <gazebo reference="p3at_front_${suffix}_axle">
-        <material value="Gazebo/Grey"/>
-    </gazebo>
-    <joint name="base_front_${suffix}_axle_joint" type="fixed">
-        <origin xyz="0.135 ${reflect*0.156} 0.111" rpy="0 0 0"/>
-        <parent link="base_link"/>
-        <child link="p3at_front_${suffix}_axle"/>
-    </joint>
-    <link name="p3at_front_${suffix}_hub">
-        <inertial>
-            <mass value="0.1"/>
-            <origin xyz="0 0 0"/>
-            <inertia ixx="1.0" ixy="0.0" ixz="0.0"
-                 iyy="1.0" iyz="0.0" izz="1.0"/>
-        </inertial>
-    <visual name="base_visual">
-        <origin xyz="0 0 0" rpy="0 0 0"/>
-        <geometry name="pioneer_geom">
-            <mesh filename="package://p3at_tutorial/meshes/p3at_meshes/${suffix}_hubcap.dae"/>
-        </geometry>
-        <material name="HubcapYellow">
-            <color rgba="1.0 0.811 0.151 1.0"/>
-        </material>
-    </visual>
-    <collision>
-        <origin xyz="0 0 0" rpy="0 0 0"/>
-        <geometry>
-            <box size="0.01 0.01 0.01"/>
-        </geometry>
-    </collision>
-    </link>
-    <gazebo reference="p3at_front_${suffix}_hub">
-        <material value="Gazebo/Yellow"/>
-    </gazebo>
-    <joint name="base_front_${suffix}_hub_joint" type="fixed">
-        <origin xyz="0 ${reflect*0.041} 0" rpy="0 0 0"/>
-        <parent link="p3at_front_${suffix}_axle"/>
-        <child link="p3at_front_${suffix}_hub"/>
-    </joint>
-    <link name="p3at_front_${suffix}_wheel">
-        <inertial>
-            <mass value="0.5"/>
-            <origin xyz="0 0 0"/>
-            <inertia ixx="0.012411765597" ixy="0" ixz="0"
-         iyy="0.015218160428" iyz="0" izz="0.011763977943"/>
-      </inertial>
-    <visual name="base_visual">
-        <origin xyz="0 0 0" rpy="0 0 0"/>
-        <geometry name="pioneer_geom">
-            <mesh filename="package://p3at_tutorial/meshes/p3at_meshes/wheel.dae"/>
-        </geometry>
-        <material name="WheelBlack">
-            <color rgba="0.117 0.117 0.117 1"/>
-        </material>
-    </visual>
-    <collision>
-        <origin xyz="0 0 0" rpy="${-3.1415927/2} 0 0"/>
-        <geometry>
-        <!--mesh filename="package://p3at_tutorial/meshes/p3at_meshes/wheel.dae"/-->
-        <cylinder radius="0.111" length="0.075"/>
-        </geometry>
-    </collision>
-    </link>
-    <gazebo reference="p3at_front_${suffix}_wheel">
-        <material value="Gazebo/Black"/>
-    </gazebo>
-    <joint name="p3at_front_${suffix}_wheel_joint" type="continuous">
-    <axis xyz="0 1 0"/>
-        <anchor xyz="0 0 0"/>
-    <origin xyz="0 0 0" rpy="0 0 0"/>
-    <parent link="p3at_front_${suffix}_hub"/>
-    <child link="p3at_front_${suffix}_wheel"/>
-        <limit effort="100" velocity="100" />
-        <joint_properties damping="0.7"/>
-    </joint>
-<!-- Back Axles + Wheels + Hubcaps -->
-    <link name="p3at_back_${suffix}_axle">
-        <inertial>
-            <mass value="0.1"/>
-            <origin xyz="0 0 0"/>
-            <inertia ixx="1.0" ixy="0.0" ixz="0.0"
-                 iyy="1.0" iyz="0.0" izz="1.0"/>
-        </inertial>
-    <visual name="base_visual">
-        <origin xyz="0 0 0" rpy="0 0 0"/>
-        <geometry name="pioneer_geom">
-            <mesh filename="package://p3at_tutorial/meshes/p3at_meshes/axle.dae"/>
-        </geometry>
-        <material name="AxleGrey">
-            <color rgba="0.5 0.5 0.5 1"/>
-        </material>
-    </visual>
-    <collision>
-        <origin xyz="0 0 0" rpy="0 0 0"/>
-        <geometry>
-            <mesh filename="package://p3at_tutorial/meshes/p3at_meshes/axle.dae"/>
-        </geometry>
-    </collision>
-    </link>
-    <gazebo reference="p3at_back_${suffix}_axle">
-        <material value="Gazebo/Grey"/>
-    </gazebo>
-    <joint name="p3at_back_${suffix}_axle_joint" type="fixed">
-        <origin xyz="-0.134 ${reflect*0.156} 0.111" rpy="0 0 0"/>
-        <parent link="base_link"/>
-        <child link="p3at_back_${suffix}_axle"/>
-    </joint>
-    <link name="p3at_back_${suffix}_hub">
-        <inertial>
-            <mass value="0.1"/>
-            <origin xyz="0 0 0"/>
-            <inertia ixx="1.0" ixy="0.0" ixz="0.0"
-                 iyy="1.0" iyz="0.0" izz="1.0"/>
-        </inertial>
-    <visual name="base_visual">
-        <origin xyz="0 0 0" rpy="0 0 0"/>
-        <geometry name="pioneer_geom">
-            <mesh filename="package://p3at_tutorial/meshes/p3at_meshes/${suffix}_hubcap.dae"/>
-        </geometry>
-        <material name="HubcapYellow"/>
-    </visual>
-    <collision>
-        <origin xyz="0 0 0" rpy="0 0 0"/>
-        <geometry>
-            <mesh filename="package://p3at_tutorial/meshes/p3at_meshes/${suffix}_hubcap.dae"/>
-        </geometry>
-    </collision>
-    </link>
-    <gazebo reference="p3at_back_${suffix}_hub">
-        <material value="Gazebo/Yellow"/>
-    </gazebo>
-    <joint name="p3at_back_${suffix}_hub_joint" type="fixed">
-        <origin xyz="-0 ${reflect*0.041} 0" rpy="0 0 0"/>
-        <parent link="p3at_back_${suffix}_axle"/>
-        <child link="p3at_back_${suffix}_hub"/>
-    </joint>
-    <link name="p3at_back_${suffix}_wheel">
-        <inertial>
-            <mass value="0.5"/>
-            <origin xyz="0 0 0"/>
-            <inertia ixx="0.012411765597" ixy="0" ixz="0"
-         iyy="0.015218160428" iyz="0" izz="0.011763977943"/>
-      </inertial>
-    <visual name="base_visual">
-        <origin xyz="0 0 0" rpy="0 0 0"/>
-        <geometry name="pioneer_geom">
-            <mesh filename="package://p3at_tutorial/meshes/p3at_meshes/wheel.dae"/>
-        </geometry>
-        <material name="WheelBlack"/>
-    </visual>
-    <collision>
-        <origin xyz="0 0 0" rpy="${-3.1415927/2} 0 0"/>
-        <geometry>
-        <!--mesh filename="package://p3at_tutorial/meshes/p3at_meshes/wheel.dae"/-->
-        <cylinder radius="0.111" length="0.075"/>
-        </geometry>
-    </collision>
-    </link>
-    <gazebo reference="p3at_back_${suffix}_wheel">
-        <material value="Gazebo/Black"/>
-    </gazebo>
-    <joint name="p3at_back_${suffix}_wheel_joint" type="continuous">
-      <axis xyz="0 1 0"/>
-          <anchor xyz="0 0 0"/>
-          <limit effort="100" velocity="100" />
-          <joint_properties damping="0.7"/>
-        <origin xyz="0 0 0" rpy="0 0 0"/>
-        <parent link="p3at_back_${suffix}_hub"/>
-        <child link="p3at_back_${suffix}_wheel"/>
-    </joint>
-  <gazebo reference="p3at_back_${suffix}_wheel">
-    <kp>1000000.0</kp> <!-- kp and kd for rubber -->
-    <kd>100.0</kd>
-    <mu1>1.0</mu1>
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